File: PCBs/PowerSensingBoard/PowerSensingBoard.brd (EAGLE design)
At the start: 100 x 80 mm, 38 parts, among them IC1 7805DT, U1 ATTINY84-20SSU

Commit message: Current sensing progress
Parts:
- added J1: (no value), SparkFun-Connectors:2X03
- added J2: (no value), SparkFun-Connectors:1X02
- added SV1: (no value), con-lstb:MA04-2
- moved C17 40.9 mm to (38.1, 37.5)
- moved C10 40.2 mm to (40.6, 32.4)
- moved C11 40.2 mm to (48.3, 32.4)
- moved C12 40.2 mm to (45.7, 32.4)
- moved C9 40.2 mm to (43.2, 32.4)
- moved ADC1 39.0 mm to (24.1, 36.8)
- moved C1 39.0 mm to (9.53, 25.4)
- moved C13 39.0 mm to (35.6, 32.4)
- moved C14 39.0 mm to (38.1, 32.4)
- moved C15 39.0 mm to (32.4, 31.8)
- moved C16 39.0 mm to (40.6, 37.5)
- moved C2 39.0 mm to (19.7, 25.4)
- moved C3 39.0 mm to (29.8, 25.4)
- moved C5 39.0 mm to (50.2, 25.4)
- moved C6 39.0 mm to (60.3, 25.4)
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Connections:
- removed net N$1: U1.5
- removed net N$14: U1.6
- removed net N$16: IC1.1
- removed net N$17: IC1.3
- removed net N$6: U1.13
- removed net N$7: U1.12
- removed net N$8: U1.11
- new net 12V: IC1.1, J2.1
- new net P0: SV1.2, U1.13
- new net P1: SV1.4, U1.12
- new net P2: SV1.6, U1.11
- net 5V: now also J1.2
- net CLK: now also J1.3
- net CONVST: now also SV1.5, U1.5
- net GND: now also IC1.3, J1.6, J2.2
- net MISO: now also J1.1
- net MOSI: now also J1.4
- net RST: now also J1.5
- net RX: now also SV1.3
- net TX: now also SV1.1
- net ~BUSY: now also SV1.8
- net ~RD: now also SV1.7, U1.6
Routing:
- net 5V: track 134.9 -> 124.9 mm
- net A7: track 90.0 -> 85.9 mm
- net A1: track 40.5 -> 38.3 mm
- net A2: track 48.8 -> 46.5 mm
- net A3: track 57.0 -> 54.8 mm
- net A4: track 65.3 -> 63.0 mm
- net A5: track 73.5 -> 71.3 mm
- net A6: track 81.7 -> 79.5 mm
- net N$11: track 16.2 -> 17.4 mm
- net A0: track 32.3 -> 31.5 mm
- added copper zone on layer 16, net GND
Other:
- board size 100 x 80 mm -> 100 x 49.5 mm

Commit message: Sensing board progress
Parts:
- moved C14 5.91 mm to (32.4, 33.9), turned to 180 degrees
- moved C16 5.08 mm to (35.6, 37.5)
- moved C17 5.08 mm to (33.0, 37.5)
- moved C12 3.81 mm to (41.9, 32.4)
- moved C10 3.17 mm to (37.5, 32.4)
- moved C9 3.17 mm to (40.0, 32.4)
- moved C11 2.54 mm to (45.7, 32.4)
- moved C15 1.27 mm to (31.1, 31.8)
- moved C13 0.64 mm to (34.9, 32.4)
Routing:
- net CONVST: track 0.00 -> 61.4 mm, vias 0 -> 1
- net P0: track 0.00 -> 59.4 mm
- net CLK: track 0.00 -> 55.0 mm, vias 0 -> 2
- net ~BUSY: track 0.00 -> 54.1 mm, vias 0 -> 2
- net ~RD: track 0.00 -> 52.6 mm, vias 0 -> 1
- net MISO: track 0.00 -> 52.5 mm, vias 0 -> 3
- net MOSI: track 0.00 -> 47.2 mm, vias 0 -> 3
- net 5V: track 124.9 -> 166.1 mm, vias 0 -> 3
- net TX: track 0.00 -> 28.7 mm
- net P1: track 0.00 -> 26.5 mm
- net RX: track 0.00 -> 25.4 mm
- net P2: track 0.00 -> 23.1 mm
- net RST: track 0.00 -> 12.6 mm
- net 12V: track 0.00 -> 7.45 mm
- net N$11: track 17.4 -> 13.2 mm
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