File: PCBs/PowerSensingBoard/PowerSensingBoard.brd (EAGLE design)
At the start: 100 x 49.5 mm, 41 parts, among them IC1 7805DT, U1 ATTINY84-20SSU

Commit message: Moved stuff around
Parts:
- removed J2: (no value), SparkFun-Connectors:1X02
- added X9: (no value), con-wago-500:W237-102
- moved IC1 22.3 mm to (93.3, 17.1), turned to 180 degrees
- moved C16 7.24 mm to (42.5, 35.6)
- moved C17 7.24 mm to (40.0, 35.6)
- moved CSENSE6 4.84 mm to (73.0, 17.1)
- moved CSENSE7 4.84 mm to (83.2, 17.1)
- moved SV1 4.84 mm to (83.2, 32.4)
- moved X7 4.84 mm to (73.0, 9.53)
- moved X8 4.84 mm to (83.2, 9.53)
- moved C7 4.84 mm to (74.9, 23.5)
- moved C8 4.84 mm to (85.1, 23.5)
- moved C15 4.84 mm to (35.6, 29.8)
- moved J1 4.84 mm to (74.3, 40.0)
- moved ADC1 4.84 mm to (28.6, 34.9)
- moved C14 4.84 mm to (36.8, 32.0)
- moved CSENSE1 4.84 mm to (22.2, 17.1)
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Connections:
- net 12V: now also X9.1; no longer J2.1
- net GND: now also X9.2; no longer J2.2
Routing:
- net CLK: track 55.0 -> 57.9 mm
- net 5V: track 166.1 -> 168.5 mm
- net MISO: track 52.5 -> 53.9 mm
- net CONVST: track 61.4 -> 62.2 mm
- net 12V: track 7.45 -> 6.72 mm
- net ~BUSY: track 54.1 -> 54.7 mm
- net MOSI: track 47.2 -> 47.7 mm, vias 3 -> 1
Other:
- board size 100 x 49.5 mm -> 100 x 45.7 mm

Commit message: Made berbers for Sensing and power bus boards
Parts:
- added C18, C19, C21: 4.7uF, SparkFun-Capacitors:0603-CAP
- added C20: 0.33uF, SparkFun-Capacitors:0805-CAP
- added LED1: (no value), adafruit:CHIP-LED0805
- added R3: 10k, SparkFun-Resistors:0805
- added R4: 100, SparkFun-Resistors:0603-RES
- moved IC1 87.8 mm to (5.71, 22.9), turned to 0 degrees
- moved X9 87.7 mm to (5.08, 33.7), turned to 270 degrees
- moved C12 1.91 mm to (48.3, 30.5)
- moved C10 1.27 mm to (43.2, 30.5)
- moved C11 1.27 mm to (51.4, 30.5)
- moved C13 1.27 mm to (40.6, 30.5)
- moved C9 1.27 mm to (45.7, 30.5)
- moved SV1 1.27 mm to (81.9, 32.4)
- renumbered J1 to ISP
Connections:
- net N$2 renamed MUXOUT+
- net N$3 renamed MUXOUT-
- net P0 renamed PA0
- net P1 renamed PA1
- net P2 renamed PA2
- removed net N$4: U1.14
- new net LED1: LED1.C, R4.2
- net 12V: now also C19.1
- net 5V: now also C18.1, C21.1, LED1.A, R3.1
- net GND: now also C18.2, C19.2, C20.2, C21.2, R4.1, U1.14
- net RST: now also C20.1, R3.2
Routing:
- net PA0: track 59.4 -> 25.3 mm, vias 0 -> 1
- net 12V: track 6.72 -> 33.2 mm, vias 0 -> 4
- net GND: track 0.00 -> 19.8 mm, vias 16 -> 151
- net 5V: track 168.5 -> 185.3 mm, vias 3 -> 4
- net RST: track 12.4 -> 16.0 mm, vias 0 -> 1
- net PA1: track 26.5 -> 24.5 mm
- net LED1: track 0.00 -> 1.99 mm
- net RX: track 25.4 -> 23.5 mm
- net TX: track 28.3 -> 26.7 mm
- net N$13: track 9.04 -> 10.3 mm
- net ~RD: track 52.6 -> 51.3 mm
- net N$11: track 13.2 -> 14.5 mm
- net MISO: track 53.9 -> 55.2 mm
- net N$10: track 19.3 -> 20.4 mm
- net ~BUSY: track 54.7 -> 55.5 mm
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Other:
- board size 100 x 45.7 mm -> 97.5 x 45.7 mm
- board text added: "+ A1 -"
- board text added: "+ A2 -"
- board text added: "+ M1 -"
- board text added: "+ M2 -"
- board text added: "+ M3 -"
- board text added: "+ M4 -"
- board text added: "+ M5 -"
- board text added: "+ M6 -"
- board text added: "Andrew Hostler"
- board text added: "Power"
- board text added: "UROV Power Sensing Board v 1.0"
- board text added: "~BSY PA2 PA1 PA0"
- board text added: "~RD CVST RX TX"
