File: PCBs/PowerSensingBoard/PowerSensingBoard2.brd (EAGLE design)
At the start: 100 x 45.7 mm, 41 parts, among them IC1 7805DT, U1 ATTINY84-20SSU

Commit message: Moved stuff around
Parts:
- moved X9 101.4 mm to (92.7, 30.5), turned to 90 degrees
- moved IC1 3.81 mm to (93.3, 17.1)
- moved C9 0.25 mm to (44.2, 30.5)
Connections:
- net 12V: now also X9.1
- net GND: now also X9.2
Routing:
- net MISO: track 53.0 -> 53.9 mm, vias 1 -> 3
