File: PCBs/PowerSensingBoard/PowerSensingBoard.sch (EAGLE design)
At the start: 41 parts, among them IC1 7805DT, U1 ATTINY84-20SSU

Commit message: Made berbers for Sensing and power bus boards
Parts:
- added C18, C19, C21: 4.7uF, SparkFun-Capacitors:4.7UF-6.3V-10%(0603)0603
- added C20: 0.33uF, SparkFun-Capacitors:0.33UF-50V-10%(0805)
- added LED1: (no value), adafruit:LEDCHIP-LED0805
- added R3: 10k, SparkFun-Resistors:0.3OHM-1/8W-1%(0805)
- added R4: 100, SparkFun-Resistors:1KOHM-1/10W-1%(0603)
- renumbered J1 to ISP
Connections:
- net N$2 renamed MUXOUT+
- net N$3 renamed MUXOUT-
- net P0 renamed PA0
- net P1 renamed PA1
- net P2 renamed PA2
- removed net N$4: U1.GND
- new net LED1: LED1.C, R4.2
- net 12V: now also C19.1
- net 5V: now also C18.1, C21.1, LED1.A, R3.1
- net GND: now also C18.2, C19.2, C20.2, C21.2, R4.1, U1.GND
- net RST: now also C20.1, R3.2
Other:
- moved on the sheet: IC1, X9-1, X9-2
