File: PCBs/Comms Board/urov schematic_2.sch (EAGLE design)
At the start: 24 parts

Commit message: Comms board edits
Parts:
- removed SL1: (no value), con-amp-quick:M02
- removed SL2: (no value), con-amp-quick:M08
- removed SL3: (no value), con-amp-quick:M04
- removed U$3: ATTINY84ATTINY84-20PU, SparkFun-DigitalIC:ATTINY84ATTINY84-20PU
Changed lines of the file:
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@@
 <part name="J13" library="SparkFun-Connectors" deviceset="M04" device="PTH"/>
 <part name="J14" library="SparkFun-Connectors" deviceset="M02" device="PTH"/>
-<part name="U$3" library="SparkFun-DigitalIC" deviceset="ATTINY84" device="ATTINY84-20PU"/>
-<part name="SL1" library="con-amp-quick" deviceset="M02" device=""/>
-<part name="SL2" library="con-amp-quick" deviceset="M08" device=""/>
-<part name="SL3" library="con-amp-quick" deviceset="M04" device=""/>
 <part name="U$4" library="UROV_Accessories" deviceset="MAX4574" device="A"/>
 </parts>
@@
 <instance part="J13" gate="G$1" x="-182.88" y="50.8"/>
 <instance part="J14" gate="G$1" x="-157.48" y="33.02"/>
-<instance part="U$3" gate="G$1" x="-5.08" y="137.16"/>
-<instance part="SL1" gate="G$1" x="-40.64" y="134.62"/>
-<instance part="SL2" gate="G$1" x="30.48" y="132.08" rot="R180"/>
-<instance part="SL3" gate="G$1" x="30.48" y="149.86" rot="R180"/>
 <instance part="U$4" gate="G$1" x="5.08" y="83.82"/>
 </instances>
