File: PCBs/Comms Board/urov schematic_2.brd (EAGLE design)
At the start: 100 x 80 mm, 18 parts

Commit message: Adding jumpers to select I2C or SPI
Parts:
- added J14: (no value), SparkFun-Connectors:1X02
- moved J13 47.1 mm to (44.5, 12.7)
- moved J12 11.7 mm to (10.2, 5.08)
Connections:
- net MOSI: now also J12.1
- net SCL: now also J14.2
- net SCLK: now also J14.1
- net SDA: now also J12.2
Changed lines of the file:
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@@
 <attribute name="PROD_ID" value="CONN-09696" x="5.08" y="15.24" size="1.778" layer="27" display="off"/>
 </element>
-<element name="J12" library="SparkFun-Connectors" package="1X02" value="" x="2.54" y="-3.81"/>
+<element name="J12" library="SparkFun-Connectors" package="1X02" value="" x="10.16" y="5.08"/>
 <element name="PRESSURE_INTERNAL" library="SparkFun-Sensors" package="MS5803" value="MS5803-14BA" x="59.69" y="27.94">
 <attribute name="PROD_ID" value="IC-12111" x="59.69" y="27.94" size="1.778" layer="27" display="off"/>
 </element>
-<element name="J13" library="SparkFun-Connectors" package="1X04" value="" x="2.54" y="-8.89">
-<attribute name="PROD_ID" value="CONN-09696" x="2.54" y="-8.89" size="1.778" layer="27" display="off"/>
+<element name="J13" library="SparkFun-Connectors" package="1X04" value="" x="44.45" y="12.7">
+<attribute name="PROD_ID" value="CONN-09696" x="44.45" y="12.7" size="1.778" layer="27" display="off"/>
 </element>
+<element name="J14" library="SparkFun-Connectors" package="1X02" value="" x="29.21" y="13.97" rot="R180"/>
 </elements>
 <signals>
@@
 <contactref element="J11" pad="4"/>
 <contactref element="PRESSURE_INTERNAL" pad="1"/>
+<contactref element="J14" pad="2"/>
 <wire x1="12.7" y1="15.24" x2="57.015" y2="29.84" width="0" layer="19" extent="1-1"/>
+<wire x1="26.67" y1="13.97" x2="12.7" y2="15.24" width="0" layer="19" extent="1-1"/>
 </signal>
 <signal name="SDA">
 <contactref element="J11" pad="3"/>
+<contactref element="J12" pad="2"/>
+<wire x1="12.7" y1="5.08" x2="10.16" y2="15.24" width="0" layer="19" extent="1-1"/>
 </signal>
 <signal name="VDD_9DOF_3.3V">
@@
 <contactref element="PRESSURE_INTERNAL" pad="8"/>
 <contactref element="J13" pad="3"/>
-<wire x1="7.62" y1="-8.89" x2="62.365" y2="29.84" width="0" layer="19" extent="1-1"/>
+<wire x1="49.53" y1="12.7" x2="62.365" y2="29.84" width="0" layer="19" extent="1-1"/>
 </signal>
 <signal name="V3.3">
@@
 <contactref element="PRESSURE_INTERNAL" pad="7"/>
 <contactref element="J13" pad="4"/>
-<wire x1="10.16" y1="-8.89" x2="62.365" y2="28.59" width="0" layer="19" extent="1-1"/>
+<contactref element="J12" pad="1"/>
+<wire x1="52.07" y1="12.7" x2="62.365" y2="28.59" width="0" layer="19" extent="1-1"/>
+<wire x1="10.16" y1="5.08" x2="52.07" y2="12.7" width="0" layer="19" extent="1-1"/>
 </signal>
 <signal name="SCLK">
 <contactref element="J13" pad="2"/>
+<contactref element="J14" pad="1"/>
+<wire x1="29.21" y1="13.97" x2="46.99" y2="12.7" width="0" layer="19" extent="1-1"/>
 </signal>
 <signal name="SS">
 <contactref element="J13" pad="1"/>
 <contactref element="PRESSURE_INTERNAL" pad="3"/>
-<wire x1="2.54" y1="-8.89" x2="57.29" y2="27.29" width="0" layer="19" extent="1-1"/>
+<wire x1="44.45" y1="12.7" x2="57.29" y2="27.29" width="0" layer="19" extent="1-1"/>
 </signal>
 </signals>

Commit message: added ATTTINY84 and headers
started working on creating MAX4574 from scratch
Parts:
- added SL1: (no value), con-amp-quick:02P
- added SL2: (no value), con-amp-quick:08P
- added SL3: (no value), con-amp-quick:04P
- added U$3: ATTINY84ATTINY84-20PU, SparkFun-DigitalIC:DIL14
Changed lines of the file:
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@@
 </element>
 <element name="J14" library="SparkFun-Connectors" package="1X02" value="" x="29.21" y="13.97" rot="R180"/>
+<element name="U$3" library="SparkFun-DigitalIC" package="DIL14" value="ATTINY84ATTINY84-20PU" x="11.43" y="-6.35"/>
+<element name="SL1" library="con-amp-quick" package="02P" value="" x="-5.08" y="-7.62">
+<attribute name="MF" value="" x="-5.08" y="-7.62" size="1.778" layer="27" display="off"/>
+<attribute name="OC_NEWARK" value="unknown" x="-5.08" y="-7.62" size="1.778" layer="27" display="off"/>
+<attribute name="MPN" value="" x="-5.08" y="-7.62" size="1.778" layer="27" display="off"/>
+<attribute name="OC_FARNELL" value="unknown" x="-5.08" y="-7.62" size="1.778" layer="27" display="off"/>
+</element>
+<element name="SL2" library="con-amp-quick" package="08P" value="" x="2.54" y="-17.78">
+<attribute name="MF" value="" x="2.54" y="-17.78" size="1.778" layer="27" display="off"/>
+<attribute name="OC_NEWARK" value="unknown" x="2.54" y="-17.78" size="1.778" layer="27" display="off"/>
+<attribute name="MPN" value="" x="2.54" y="-17.78" size="1.778" layer="27" display="off"/>
+<attribute name="OC_FARNELL" value="unknown" x="2.54" y="-17.78" size="1.778" layer="27" display="off"/>
+</element>
+<element name="SL3" library="con-amp-quick" package="04P" value="" x="-2.54" y="-25.4">
+<attribute name="MF" value="" x="-2.54" y="-25.4" size="1.778" layer="27" display="off"/>
+<attribute name="OC_NEWARK" value="unknown" x="-2.54" y="-25.4" size="1.778" layer="27" display="off"/>
+<attribute name="MPN" value="" x="-2.54" y="-25.4" size="1.778" layer="27" display="off"/>
+<attribute name="OC_FARNELL" value="unknown" x="-2.54" y="-25.4" size="1.778" layer="27" display="off"/>
+</element>
 </elements>
 <signals>

Commit message: added max4574
took forever
Parts:
- added U$4: MAX4574A, UROV_Accessories:28-SSOP
Changed lines of the file:
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@@
 <attribute name="OC_FARNELL" value="unknown" x="-2.54" y="-25.4" size="1.778" layer="27" display="off"/>
 </element>
+<element name="U$4" library="UROV_Accessories" package="28-SSOP" value="MAX4574A" x="0" y="-33.02"/>
 </elements>
 <signals>

Commit message: Comms board edits
Parts:
- removed SL1: (no value), con-amp-quick:02P
- removed SL2: (no value), con-amp-quick:08P
- removed SL3: (no value), con-amp-quick:04P
- removed U$3: ATTINY84ATTINY84-20PU, SparkFun-DigitalIC:DIL14
- moved U$4 103.5 mm to (77.5, 35.6)
Changed lines of the file:
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@@
 </element>
 <element name="J14" library="SparkFun-Connectors" package="1X02" value="" x="29.21" y="13.97" rot="R180"/>
-<element name="U$3" library="SparkFun-DigitalIC" package="DIL14" value="ATTINY84ATTINY84-20PU" x="11.43" y="-6.35"/>
-<element name="SL1" library="con-amp-quick" package="02P" value="" x="-5.08" y="-7.62">
-<attribute name="MF" value="" x="-5.08" y="-7.62" size="1.778" layer="27" display="off"/>
-<attribute name="OC_NEWARK" value="unknown" x="-5.08" y="-7.62" size="1.778" layer="27" display="off"/>
-<attribute name="MPN" value="" x="-5.08" y="-7.62" size="1.778" layer="27" display="off"/>
-<attribute name="OC_FARNELL" value="unknown" x="-5.08" y="-7.62" size="1.778" layer="27" display="off"/>
-</element>
-<element name="SL2" library="con-amp-quick" package="08P" value="" x="2.54" y="-17.78">
-<attribute name="MF" value="" x="2.54" y="-17.78" size="1.778" layer="27" display="off"/>
-<attribute name="OC_NEWARK" value="unknown" x="2.54" y="-17.78" size="1.778" layer="27" display="off"/>
-<attribute name="MPN" value="" x="2.54" y="-17.78" size="1.778" layer="27" display="off"/>
-<attribute name="OC_FARNELL" value="unknown" x="2.54" y="-17.78" size="1.778" layer="27" display="off"/>
-</element>
-<element name="SL3" library="con-amp-quick" package="04P" value="" x="-2.54" y="-25.4">
-<attribute name="MF" value="" x="-2.54" y="-25.4" size="1.778" layer="27" display="off"/>
-<attribute name="OC_NEWARK" value="unknown" x="-2.54" y="-25.4" size="1.778" layer="27" display="off"/>
-<attribute name="MPN" value="" x="-2.54" y="-25.4" size="1.778" layer="27" display="off"/>
-<attribute name="OC_FARNELL" value="unknown" x="-2.54" y="-25.4" size="1.778" layer="27" display="off"/>
-</element>
-<element name="U$4" library="UROV_Accessories" package="28-SSOP" value="MAX4574A" x="0" y="-33.02"/>
+<element name="U$4" library="UROV_Accessories" package="28-SSOP" value="MAX4574A" x="77.47" y="35.56"/>
 </elements>
 <signals>

Commit message: Made berbers for Sensing and power bus boards
Parts:
- moved J14 10.5 mm to (31.8, 3.81)
Routing:
- net A_DIP8_1: track 21.2 -> 20.4 mm
Changed lines of the file:
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@@
 <attribute name="PROD_ID" value="CONN-09696" x="44.45" y="12.7" size="1.778" layer="27" display="off"/>
 </element>
-<element name="J14" library="SparkFun-Connectors" package="1X02" value="" x="29.21" y="13.97" rot="R180"/>
+<element name="J14" library="SparkFun-Connectors" package="1X02" value="" x="31.75" y="3.81" rot="R180"/>
 <element name="U$4" library="UROV_Accessories" package="28-SSOP" value="MAX4574A" x="77.47" y="35.56"/>
 </elements>
@@
 <wire x1="8.52" y1="27.94" x2="8.89" y2="27.57" width="0.4064" layer="1"/>
 <wire x1="8.89" y1="27.57" x2="9.26" y2="27.94" width="0.4064" layer="1"/>
-<wire x1="9.26" y1="27.94" x2="15.24" y2="27.94" width="0.4064" layer="1"/>
-<wire x1="15.24" y1="27.94" x2="15.24" y2="34.29" width="0.4064" layer="1"/>
+<wire x1="9.26" y1="27.94" x2="13.97" y2="27.94" width="0.4064" layer="1"/>
+<wire x1="13.97" y1="27.94" x2="15.24" y2="29.21" width="0.4064" layer="1"/>
+<wire x1="15.24" y1="29.21" x2="15.24" y2="34.29" width="0.4064" layer="1"/>
 <wire x1="15.24" y1="34.29" x2="16.51" y2="35.56" width="0.4064" layer="1"/>
 <wire x1="16.51" y1="35.56" x2="19.05" y2="35.56" width="0.4064" layer="1"/>
@@
 <contactref element="J14" pad="2"/>
 <wire x1="12.7" y1="15.24" x2="57.015" y2="29.84" width="0" layer="19" extent="1-1"/>
-<wire x1="26.67" y1="13.97" x2="12.7" y2="15.24" width="0" layer="19" extent="1-1"/>
+<wire x1="29.21" y1="3.81" x2="12.7" y2="15.24" width="0" layer="19" extent="1-1"/>
 </signal>
 <signal name="SDA">
@@
 <contactref element="J13" pad="2"/>
 <contactref element="J14" pad="1"/>
-<wire x1="29.21" y1="13.97" x2="46.99" y2="12.7" width="0" layer="19" extent="1-1"/>
+<wire x1="31.75" y1="3.81" x2="46.99" y2="12.7" width="0" layer="19" extent="1-1"/>
 </signal>
 <signal name="SS">
