File: PCBs/Comms Board/urov schematic_3.brd (EAGLE design)
At the start: 100 x 80 mm, 24 parts

Commit message: Accessory Board possible edits
Unless Josh had better changes
Parts:
- moved U$4 82.1 mm to (67.3, 14.0), turned to 270 degrees
- moved U$3 77.3 mm to (80.0, 29.2), turned to 270 degrees
- moved SL1 61.9 mm to (54.6, 8.89)
- moved SL3 41.0 mm to (17.8, 10.2)
- moved SL2 38.4 mm to (34.3, 3.81)
- moved J7 6.48 mm to (71.1, 66.0)
- moved J1 6.48 mm to (6.35, 66.0)
- moved J2 6.48 mm to (21.6, 66.0)
- moved J3 6.48 mm to (27.9, 66.0)
- moved J4 6.48 mm to (43.2, 66.0)
- moved J5 6.48 mm to (49.5, 66.0)
- moved J6 6.48 mm to (64.8, 66.0)
- moved J8 6.48 mm to (86.4, 66.0)
Other:
- board size 100 x 80 mm -> 100 x 72.4 mm
