File: PCBs/PowerSupplyBoard/Power Supply Board.brd (EAGLE design)
At the start: 99.1 x 79.8 mm, 24 parts

Commit message: Power board edits
Parts:
- SV1, SV2, SV3, SV4: device con-lstb:MA03-1 -> con-lstb:MA04-1
- moved SV2 1.27 mm to (10.2, 21.0)
- moved SV4 1.27 mm to (89.5, 23.5)
- moved SV1 1.27 mm to (10.2, 55.9)
- moved SV3 1.27 mm to (90.2, 57.8)
Connections:
- removed net N$1: SV1.3, VC1.TM, VC1.TM@1
- removed net N$10: SV4.3, VC4.TM, VC4.TM@1
- removed net N$12: SV4.1, VC4.PC, VC4.PC21
- removed net N$3: SV1.1, VC1.PC, VC1.PC21
- removed net N$4: SV2.3, VC2.TM, VC2.TM@1
- removed net N$6: SV2.1, VC2.PC, VC2.PC21
- removed net N$7: SV3.3, VC3.TM, VC3.TM@1
- removed net N$9: SV3.1, VC3.PC, VC3.PC21
- new net PC1: SV1.1, SV1.2, VC1.PC, VC1.PC21
- new net PC2: SV2.1, SV2.2, VC2.PC, VC2.PC21
- new net PC3: SV3.1, SV3.2, VC3.PC, VC3.PC21
- new net PC4: SV4.1, SV4.2, VC4.PC, VC4.PC21
- new net TM1: SV1.4, VC1.TM, VC1.TM@1
- new net TM2: SV2.4, VC2.TM, VC2.TM@1
- new net TM3: SV3.4, VC3.TM, VC3.TM@1
- new net TM4: SV4.4, VC4.TM, VC4.TM@1
- net N$11: now also SV4.3; no longer SV4.2
- net N$2: now also SV1.3; no longer SV1.2
- net N$5: now also SV2.3; no longer SV2.2
- net N$8: now also SV3.3; no longer SV3.2
Routing:
- net PC2: track 0.00 -> 10.6 mm
- net PC1: track 0.00 -> 10.6 mm
- net PC3: track 0.00 -> 10.3 mm
- net PC4: track 0.00 -> 9.70 mm
- net N$6: track 8.06 -> 0.00 mm
- net N$3: track 8.06 -> 0.00 mm
- net TM3: track 0.00 -> 8.00 mm
- net N$7: track 8.00 -> 0.00 mm
- net N$9: track 7.79 -> 0.00 mm
- net TM2: track 0.00 -> 7.73 mm
- net N$4: track 7.73 -> 0.00 mm
- net TM1: track 0.00 -> 7.73 mm
- net N$1: track 7.73 -> 0.00 mm
- net TM4: track 0.00 -> 7.36 mm
- net N$10: track 7.36 -> 0.00 mm
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
Commit message: Made berbers for Sensing and power bus boards
Parts:
- removed U$2: MOLEXMEGAFIT, MolexMegaFIT 2circuit:MOLEXMEGAFIT
- added X10, X8, X9: (no value), con-wago-500:W237-102
- moved C2 14.0 mm to (54.6, 65.4)
- moved C6 10.9 mm to (54.6, 57.8)
- moved X7 2.84 mm to (43.8, 48.9), turned to 90 degrees
- moved SV1 1.27 mm to (10.2, 57.1)
- moved U$3 0.63 mm to (4.45, 47.6)
- moved U$9 0.63 mm to (95.9, 47.6)
Connections:
- net GROUNDOUT: now also X10.2, X8.2, X9.2; no longer U$2.GRD1
- net POWEROUT: now also X10.1, X8.1, X9.1; no longer U$2.POW1
Routing:
- net TM1: track 7.73 -> 8.26 mm
Other:
- board text added: "+"
- board text added: "-"
- board text added: "Cal Poly UROV Power Board V1.2"
- board text removed: "Cal Poly UROV Power Board V1.0"
