File: PCBs/PowerSupplyBoard/Power Supply Board.sch (EAGLE design)
At the start: 24 parts

Commit message: Power board edits
Parts:
- SV1, SV2, SV3, SV4: device con-lstb:MA03-1 -> con-lstb:MA04-1
Connections:
- removed net N$1: SV1.3, VC1.TM
- removed net N$10: SV4.3, VC4.TM
- removed net N$12: SV4.1, VC4.PC
- removed net N$3: SV1.1, VC1.PC
- removed net N$4: SV2.3, VC2.TM
- removed net N$6: SV2.1, VC2.PC
- removed net N$7: SV3.3, VC3.TM
- removed net N$9: SV3.1, VC3.PC
- new net PC1: SV1.1, SV1.2, VC1.PC
- new net PC2: SV2.1, SV2.2, VC2.PC
- new net PC3: SV3.1, SV3.2, VC3.PC
- new net PC4: SV4.1, SV4.2, VC4.PC
- new net TM1: SV1.4, VC1.TM
- new net TM2: SV2.4, VC2.TM
- new net TM3: SV3.4, VC3.TM
- new net TM4: SV4.4, VC4.TM
- net N$11: now also SV4.3; no longer SV4.2
- net N$2: now also SV1.3; no longer SV1.2
- net N$5: now also SV2.3; no longer SV2.2
- net N$8: now also SV3.3; no longer SV3.2
Changed lines of the file:
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@@
 <part name="X6" library="con-wago-500" deviceset="W237-102" device=""/>
 <part name="X7" library="con-wago-500" deviceset="W237-102" device=""/>
-<part name="SV1" library="con-lstb" deviceset="MA03-1" device=""/>
-<part name="SV2" library="con-lstb" deviceset="MA03-1" device=""/>
-<part name="SV3" library="con-lstb" deviceset="MA03-1" device=""/>
-<part name="SV4" library="con-lstb" deviceset="MA03-1" device=""/>
+<part name="SV1" library="con-lstb" deviceset="MA04-1" device=""/>
+<part name="SV2" library="con-lstb" deviceset="MA04-1" device=""/>
+<part name="SV3" library="con-lstb" deviceset="MA04-1" device=""/>
+<part name="SV4" library="con-lstb" deviceset="MA04-1" device=""/>
 <part name="C3" library="capacitor-wima" deviceset="C" device="2,5-3"/>
 <part name="C4" library="capacitor-wima" deviceset="C" device="2,5-3"/>
@@
 <instance part="X7" gate="-1" x="127" y="91.44" rot="R270"/>
 <instance part="X7" gate="-2" x="132.08" y="91.44" rot="R270"/>
-<instance part="SV1" gate="G$1" x="15.24" y="-15.24" rot="R90"/>
-<instance part="SV2" gate="G$1" x="58.42" y="-15.24" rot="R90"/>
-<instance part="SV3" gate="G$1" x="101.6" y="-15.24" rot="R90"/>
-<instance part="SV4" gate="G$1" x="144.78" y="-15.24" rot="R90"/>
+<instance part="SV1" gate="1" x="15.24" y="-15.24" rot="R90"/>
+<instance part="SV2" gate="1" x="58.42" y="-15.24" rot="R90"/>
+<instance part="SV3" gate="1" x="101.6" y="-15.24" rot="R90"/>
+<instance part="SV4" gate="1" x="144.78" y="-15.24" rot="R90"/>
 <instance part="C3" gate="G$1" x="15.24" y="-27.94" rot="R90"/>
 <instance part="C4" gate="G$1" x="101.6" y="-27.94" rot="R90"/>
@@
 </segment>
 </net>
-<net name="N$1" class="0">
-<segment>
-<pinref part="SV1" gate="G$1" pin="3"/>
+<net name="TM1" class="0">
+<segment>
+<pinref part="SV1" gate="1" pin="4"/>
 <pinref part="VC1" gate="G$1" pin="TM"/>
 <wire x1="12.7" y1="-7.62" x2="12.7" y2="-5.08" width="0.1524" layer="91"/>
@@
 <net name="N$2" class="0">
 <segment>
-<pinref part="SV1" gate="G$1" pin="2"/>
+<pinref part="SV1" gate="1" pin="3"/>
 <pinref part="VC1" gate="G$1" pin="RSV"/>
 <wire x1="15.24" y1="-7.62" x2="15.24" y2="-5.08" width="0.1524" layer="91"/>
 </segment>
 </net>
-<net name="N$3" class="0">
-<segment>
-<pinref part="SV1" gate="G$1" pin="1"/>
+<net name="PC1" class="0">
+<segment>
+<pinref part="SV1" gate="1" pin="2"/>
 <pinref part="VC1" gate="G$1" pin="PC"/>
 <wire x1="17.78" y1="-7.62" x2="17.78" y2="-5.08" width="0.1524" layer="91"/>
-</segment>
-</net>
-<net name="N$4" class="0">
-<segment>
-<pinref part="SV2" gate="G$1" pin="3"/>
+<wire x1="17.78" y1="-5.08" x2="20.32" y2="-5.08" width="0.1524" layer="91"/>
+<junction x="17.78" y="-5.08"/>
+<pinref part="SV1" gate="1" pin="1"/>
+<wire x1="20.32" y1="-5.08" x2="20.32" y2="-7.62" width="0.1524" layer="91"/>
+</segment>
+</net>
+<net name="TM2" class="0">
+<segment>
+<pinref part="SV2" gate="1" pin="4"/>
 <pinref part="VC2" gate="G$1" pin="TM"/>
 <wire x1="55.88" y1="-7.62" x2="55.88" y2="-5.08" width="0.1524" layer="91"/>
@@
 <net name="N$5" class="0">
 <segment>
-<pinref part="SV2" gate="G$1" pin="2"/>
+<pinref part="SV2" gate="1" pin="3"/>
 <pinref part="VC2" gate="G$1" pin="RSV"/>
 <wire x1="58.42" y1="-7.62" x2="58.42" y2="-5.08" width="0.1524" layer="91"/>
 </segment>
 </net>
-<net name="N$6" class="0">
-<segment>
-<pinref part="SV2" gate="G$1" pin="1"/>
+<net name="PC2" class="0">
+<segment>
+<pinref part="SV2" gate="1" pin="2"/>
 <pinref part="VC2" gate="G$1" pin="PC"/>
 <wire x1="60.96" y1="-7.62" x2="60.96" y2="-5.08" width="0.1524" layer="91"/>
-</segment>
-</net>
-<net name="N$7" class="0">
+<wire x1="60.96" y1="-5.08" x2="63.5" y2="-5.08" width="0.1524" layer="91"/>
+<junction x="60.96" y="-5.08"/>
+<pinref part="SV2" gate="1" pin="1"/>
+<wire x1="63.5" y1="-5.08" x2="63.5" y2="-7.62" width="0.1524" layer="91"/>
+</segment>
+</net>
+<net name="TM3" class="0">
 <segment>
 <pinref part="VC3" gate="G$1" pin="TM"/>
-<pinref part="SV3" gate="G$1" pin="3"/>
+<pinref part="SV3" gate="1" pin="4"/>
 <wire x1="99.06" y1="-5.08" x2="99.06" y2="-7.62" width="0.1524" layer="91"/>
 </segment>
@@
 <segment>
 <pinref part="VC3" gate="G$1" pin="RSV"/>
-<pinref part="SV3" gate="G$1" pin="2"/>
+<pinref part="SV3" gate="1" pin="3"/>
 <wire x1="101.6" y1="-5.08" x2="101.6" y2="-7.62" width="0.1524" layer="91"/>
 </segment>
 </net>
-<net name="N$9" class="0">
+<net name="PC3" class="0">
 <segment>
 <pinref part="VC3" gate="G$1" pin="PC"/>
-<pinref part="SV3" gate="G$1" pin="1"/>
+<pinref part="SV3" gate="1" pin="2"/>
 <wire x1="104.14" y1="-5.08" x2="104.14" y2="-7.62" width="0.1524" layer="91"/>
-</segment>
-</net>
-<net name="N$10" class="0">
+<wire x1="104.14" y1="-5.08" x2="106.68" y2="-5.08" width="0.1524" layer="91"/>
+<junction x="104.14" y="-5.08"/>
+<pinref part="SV3" gate="1" pin="1"/>
+<wire x1="106.68" y1="-5.08" x2="106.68" y2="-7.62" width="0.1524" layer="91"/>
+</segment>
+</net>
+<net name="TM4" class="0">
 <segment>
 <pinref part="VC4" gate="G$1" pin="TM"/>
-<pinref part="SV4" gate="G$1" pin="3"/>
+<pinref part="SV4" gate="1" pin="4"/>
 <wire x1="142.24" y1="-5.08" x2="142.24" y2="-7.62" width="0.1524" layer="91"/>
 </segment>
@@
 <segment>
 <pinref part="VC4" gate="G$1" pin="RSV"/>
-<pinref part="SV4" gate="G$1" pin="2"/>
+<pinref part="SV4" gate="1" pin="3"/>
 <wire x1="144.78" y1="-5.08" x2="144.78" y2="-7.62" width="0.1524" layer="91"/>
 </segment>
 </net>
-<net name="N$12" class="0">
+<net name="PC4" class="0">
 <segment>
 <pinref part="VC4" gate="G$1" pin="PC"/>
-<pinref part="SV4" gate="G$1" pin="1"/>
+<pinref part="SV4" gate="1" pin="2"/>
 <wire x1="147.32" y1="-5.08" x2="147.32" y2="-7.62" width="0.1524" layer="91"/>
-</segment>
-</net>
+<wire x1="147.32" y1="-5.08" x2="149.86" y2="-5.08" width="0.1524" layer="91"/>
+<junction x="147.32" y="-5.08"/>
+<pinref part="SV4" gate="1" pin="1"/>
+<wire x1="149.86" y1="-5.08" x2="149.86" y2="-7.62" width="0.1524" layer="91"/>
+</segment>
+</net>

Commit message: Made berbers for Sensing and power bus boards
Parts:
- removed U$2: MOLEXMEGAFIT, MolexMegaFIT 2circuit:MOLEXMEGAFIT
- added X10, X8, X9: (no value), con-wago-500:W237-102
Connections:
- net GROUNDOUT: now also X10-2.KL, X8-2.KL, X9-2.KL; no longer U$2.GRD1
- net POWEROUT: now also X10-1.KL, X8-1.KL, X9-1.KL; no longer U$2.POW1
Other:
- moved on the sheet: X7-1, X7-2
